Commit message: Removes dependency from store-gazebo

File: mobile_manipulator/boxer_custom_description/urdf/boxer.xacro (robot description, xacro)
@@ -1,5 +1,5 @@
 <?xml version="1.0"?>
 <robot name="boxer_description" xmlns:xacro="http://www.ros.org/wiki/xacro">
-	<xacro:include filename="$(find mobile_manipulator)/boxer_custom_description/urdf/materials.urdf.xacro"/>
+	<xacro:include filename="$(find robot_model)/boxer_custom_description/urdf/materials.urdf.xacro"/>
 	<xacro:macro name="boxer_description">
 		<link name="chassis_link">
@@ -12,5 +12,5 @@
 				<origin xyz="0 0 0" rpy="0 0 0" />
 				<geometry>
-					<mesh filename="package://mobile_manipulator/boxer_custom_description/meshes/chassis_link.dae" />
+					<mesh filename="package://robot_model/boxer_custom_description/meshes/chassis_link.dae" />
 				</geometry>
 				<material name="">
@@ -21,5 +21,5 @@
 				<origin xyz="0 0 0" rpy="0 0 0" />
 				<geometry>
-					<mesh filename="package://mobile_manipulator/boxer_custom_description/meshes/chassis_link.STL" />
+					<mesh filename="package://robot_model/boxer_custom_description/meshes/chassis_link.STL" />
 				</geometry>
 			</collision>
@@ -34,5 +34,5 @@
 				<origin xyz="0 0 0" rpy="0 0 0" />
 				<geometry>
-					<mesh filename="package://mobile_manipulator/boxer_custom_description/meshes/internal_link.dae" />
+					<mesh filename="package://robot_model/boxer_custom_description/meshes/internal_link.dae" />
 				</geometry>
 				<material name="Boxer_DarkGrey"/>
@@ -44,5 +44,5 @@
       <!-- (The z axis is scaled since the whole model is rotated at the joint, and collision model resolution isn't
       very smart.) -->
-      <mesh filename="package://mobile_manipulator/boxer_custom_description/meshes/internal_link.STL" />
+      <mesh filename="package://robot_model/boxer_custom_description/meshes/internal_link.STL" />
   </geometry>
 </collision>
@@ -63,5 +63,5 @@
 		<origin xyz="0 0 0" rpy="0 0 0" />
 		<geometry>
-			<mesh filename="package://mobile_manipulator/boxer_custom_description/meshes/lift_link.dae" />
+			<mesh filename="package://robot_model/boxer_custom_description/meshes/lift_link.dae" />
 		</geometry>
 		<material name="">
@@ -72,5 +72,5 @@
 		<origin xyz="0 0 0" rpy="0 0 0" />
 		<geometry>
-			<mesh filename="package://mobile_manipulator/boxer_custom_description/meshes/lift_link.STL" />
+			<mesh filename="package://robot_model/boxer_custom_description/meshes/lift_link.STL" />
 		</geometry>
 	</collision>
@@ -88,12 +88,12 @@
 		<origin xyz="0 0 0" rpy="0 0 0" />
 		<geometry>
-			<mesh filename="package://mobile_manipulator/boxer_custom_description/meshes/top_plate.stl" />
-		</geometry>
-		<material name="Boxer_DarkGrey" />
-	</visual>
-	<collision>
-		<origin xyz="0 0 0" rpy="0 0 0" />
-		<geometry>
-			<mesh filename="package://mobile_manipulator/boxer_custom_description/meshes/top_plate_collision.stl" />
+			<mesh filename="package://robot_model/boxer_custom_description/meshes/top_plate.stl" />
+		</geometry>
+		<material name="Boxer_DarkGrey" />
+	</visual>
+	<collision>
+		<origin xyz="0 0 0" rpy="0 0 0" />
+		<geometry>
+			<mesh filename="package://robot_model/boxer_custom_description/meshes/top_plate_collision.stl" />
 		</geometry>
 	</collision>
@@ -108,12 +108,12 @@
 		<origin xyz="0 0 0" rpy="0 0 0" />
 		<geometry>
-			<mesh filename="package://mobile_manipulator/boxer_custom_description/meshes/extrusion.stl" />
-		</geometry>
-		<material name="Boxer_DarkGrey" />
-	</visual>
-	<collision>
-		<origin xyz="0 0 0" rpy="0 0 0" />
-		<geometry>
-			<mesh filename="package://mobile_manipulator/boxer_custom_description/meshes/extrusion.stl" />
+			<mesh filename="package://robot_model/boxer_custom_description/meshes/extrusion.stl" />
+		</geometry>
+		<material name="Boxer_DarkGrey" />
+	</visual>
+	<collision>
+		<origin xyz="0 0 0" rpy="0 0 0" />
+		<geometry>
+			<mesh filename="package://robot_model/boxer_custom_description/meshes/extrusion.stl" />
 		</geometry>
 	</collision>
@@ -128,12 +128,12 @@
 		<origin xyz="0 0 0" rpy="0 0 0" />
 		<geometry>
-			<mesh filename="package://mobile_manipulator/boxer_custom_description/meshes/extrusion.stl" />
-		</geometry>
-		<material name="Boxer_DarkGrey" />
-	</visual>
-	<collision>
-		<origin xyz="0 0 0" rpy="0 0 0" />
-		<geometry>
-			<mesh filename="package://mobile_manipulator/boxer_custom_description/meshes/extrusion.stl" />
+			<mesh filename="package://robot_model/boxer_custom_description/meshes/extrusion.stl" />
+		</geometry>
+		<material name="Boxer_DarkGrey" />
+	</visual>
+	<collision>
+		<origin xyz="0 0 0" rpy="0 0 0" />
+		<geometry>
+			<mesh filename="package://robot_model/boxer_custom_description/meshes/extrusion.stl" />
 		</geometry>
 	</collision>
@@ -148,12 +148,12 @@
 		<origin xyz="0 0 0" rpy="0 0 0" />
 		<geometry>
-			<mesh filename="package://mobile_manipulator/boxer_custom_description/meshes/extrusion.stl" />
-		</geometry>
-		<material name="Boxer_DarkGrey" />
-	</visual>
-	<collision>
-		<origin xyz="0 0 0" rpy="0 0 0" />
-		<geometry>
-			<mesh filename="package://mobile_manipulator/boxer_custom_description/meshes/extrusion.stl" />
+			<mesh filename="package://robot_model/boxer_custom_description/meshes/extrusion.stl" />
+		</geometry>
+		<material name="Boxer_DarkGrey" />
+	</visual>
+	<collision>
+		<origin xyz="0 0 0" rpy="0 0 0" />
+		<geometry>
+			<mesh filename="package://robot_model/boxer_custom_description/meshes/extrusion.stl" />
 		</geometry>
 	</collision>
@@ -168,12 +168,12 @@
 		<origin xyz="0 0 0" rpy="0 0 0" />
 		<geometry>
-			<mesh filename="package://mobile_manipulator/boxer_custom_description/meshes/extrusion.stl" />
-		</geometry>
-		<material name="Boxer_DarkGrey" />
-	</visual>
-	<collision>
-		<origin xyz="0 0 0" rpy="0 0 0" />
-		<geometry>
-			<mesh filename="package://mobile_manipulator/boxer_custom_description/meshes/extrusion.stl" />
+			<mesh filename="package://robot_model/boxer_custom_description/meshes/extrusion.stl" />
+		</geometry>
+		<material name="Boxer_DarkGrey" />
+	</visual>
+	<collision>
+		<origin xyz="0 0 0" rpy="0 0 0" />
+		<geometry>
+			<mesh filename="package://robot_model/boxer_custom_description/meshes/extrusion.stl" />
 		</geometry>
 	</collision>
@@ -188,12 +188,12 @@
 		<origin xyz="0 0 0" rpy="0 0 0" />
 		<geometry>
-			<mesh filename="package://mobile_manipulator/boxer_custom_description/meshes/top_plate.stl" />
-		</geometry>
-		<material name="Boxer_DarkGrey" />
-	</visual>
-	<collision>
-		<origin xyz="0 0 0" rpy="0 0 0" />
-		<geometry>
-			<mesh filename="package://mobile_manipulator/boxer_custom_description/meshes/top_plate_collision.stl" />
+			<mesh filename="package://robot_model/boxer_custom_description/meshes/top_plate.stl" />
+		</geometry>
+		<material name="Boxer_DarkGrey" />
+	</visual>
+	<collision>
+		<origin xyz="0 0 0" rpy="0 0 0" />
+		<geometry>
+			<mesh filename="package://robot_model/boxer_custom_description/meshes/top_plate_collision.stl" />
 		</geometry>
 	</collision>
@@ -327,7 +327,7 @@
 <link name="base_footprint" />
 <joint name="base_footprint_joint" type="fixed">
-	<origin xyz="0 0 0.08" rpy="0 0 0" />
-	<parent link="base_footprint" />
-	<child link="base_link" />
+	<origin xyz="0 0 -0.08" rpy="0 0 0" />
+	<parent link="base_link" />
+	<child link="base_footprint" />
 </joint>
 <!-- Link for the position of the laser. -->
