Commit message: Adds shelves CAD files to remove dependency from store-gazebo #4 : comment solved

File: mobile_manipulator/models/urdf/rooms.urdf.xacro (robot description, xacro)
@@ -10,7 +10,5 @@
       <origin xyz="0 0 0" rpy="0 0 0"/>
       <geometry>
-        <!-- <mesh filename="package://boxer_gazebo/meshes/boxer_world_rooms.dae"/> -->
-        <!-- <mesh filename="package://robot_model/world/supermarket.stl"/> -->
-        <mesh filename="package://robot_model/world/supermarket_gazebo/supermarket.dae"/>
+        <mesh filename="package://mobile_manipulator/world/supermarket.dae"/>
       </geometry>
       <!-- <material name="Gray" /> -->
@@ -19,7 +17,5 @@
       <origin xyz="0 0 0" rpy="0 0 0"/>
       <geometry>
-        <!-- <mesh filename="package://boxer_gazebo/meshes/boxer_world_rooms.dae"/> -->
-        <!-- <mesh filename="package://robot_model/world/supermarket.stl"/> -->
-        <mesh filename="package://robot_model/world/supermarket_gazebo/supermarket.dae"/>
+        <mesh filename="package://mobile_manipulator/world/supermarket.dae"/>
       </geometry>
     </collision>
