Commit message: Introducing switches for control modes

File: mobile_manipulator/franka_description/robots/panda.transmission.xacro (robot description, xacro)
@@ -1,5 +1,5 @@
 <?xml version="1.0"?>
 <robot xmlns:xacro="http://www.ros.org/wiki/xacro">
-    <xacro:macro name="panda_transmission" params="robot_name load_hand">
+    <xacro:macro name="panda_transmission" params="robot_name load_hand hi:='PositionJointInterface'">
         <!-- Load Gazebo lib and set the robot namespace -->
         <gazebo>
@@ -11,8 +11,8 @@
             <type>transmission_interface/SimpleTransmission</type>
             <joint name="${robot_name}_joint1">
-                <hardwareInterface>hardware_interface/PositionJointInterface</hardwareInterface>
+                <hardwareInterface>hardware_interface/${hi}</hardwareInterface>
             </joint>
             <actuator name="${robot_name}_motor_1">
-                <hardwareInterface>hardware_interface/PositionJointInterface</hardwareInterface>
+                <hardwareInterface>hardware_interface/${hi}</hardwareInterface>
                 <mechanicalReduction>1</mechanicalReduction>
             </actuator>
@@ -21,8 +21,8 @@
             <type>transmission_interface/SimpleTransmission</type>
             <joint name="${robot_name}_joint2">
-                <hardwareInterface>hardware_interface/PositionJointInterface</hardwareInterface>
+                <hardwareInterface>hardware_interface/${hi}</hardwareInterface>
             </joint>
             <actuator name="${robot_name}_motor_2">
-                <hardwareInterface>hardware_interface/PositionJointInterface</hardwareInterface>
+                <hardwareInterface>hardware_interface/${hi}</hardwareInterface>
                 <mechanicalReduction>1</mechanicalReduction>
             </actuator>
@@ -31,8 +31,8 @@
             <type>transmission_interface/SimpleTransmission</type>
             <joint name="${robot_name}_joint3">
-                <hardwareInterface>hardware_interface/PositionJointInterface</hardwareInterface>
+                <hardwareInterface>hardware_interface/${hi}</hardwareInterface>
             </joint>
             <actuator name="${robot_name}_motor_3">
-                <hardwareInterface>hardware_interface/PositionJointInterface</hardwareInterface>
+                <hardwareInterface>hardware_interface/${hi}</hardwareInterface>
                 <mechanicalReduction>1</mechanicalReduction>
             </actuator>
@@ -41,8 +41,8 @@
             <type>transmission_interface/SimpleTransmission</type>
             <joint name="${robot_name}_joint4">
-                <hardwareInterface>hardware_interface/PositionJointInterface</hardwareInterface>
+                <hardwareInterface>hardware_interface/${hi}</hardwareInterface>
             </joint>
             <actuator name="${robot_name}_motor_4">
-                <hardwareInterface>hardware_interface/PositionJointInterface</hardwareInterface>
+                <hardwareInterface>hardware_interface/${hi}</hardwareInterface>
                 <mechanicalReduction>1</mechanicalReduction>
             </actuator>
@@ -51,8 +51,8 @@
             <type>transmission_interface/SimpleTransmission</type>
             <joint name="${robot_name}_joint5">
-                <hardwareInterface>hardware_interface/PositionJointInterface</hardwareInterface>
+                <hardwareInterface>hardware_interface/${hi}</hardwareInterface>
             </joint>
             <actuator name="${robot_name}_motor_5">
-                <hardwareInterface>hardware_interface/PositionJointInterface</hardwareInterface>
+                <hardwareInterface>hardware_interface/${hi}</hardwareInterface>
                 <mechanicalReduction>1</mechanicalReduction>
             </actuator>
@@ -61,8 +61,8 @@
             <type>transmission_interface/SimpleTransmission</type>
             <joint name="${robot_name}_joint6">
-                <hardwareInterface>hardware_interface/PositionJointInterface</hardwareInterface>
+                <hardwareInterface>hardware_interface/${hi}</hardwareInterface>
             </joint>
             <actuator name="${robot_name}_motor_6">
-                <hardwareInterface>hardware_interface/PositionJointInterface</hardwareInterface>
+                <hardwareInterface>hardware_interface/${hi}</hardwareInterface>
                 <mechanicalReduction>1</mechanicalReduction>
             </actuator>
@@ -71,8 +71,8 @@
             <type>transmission_interface/SimpleTransmission</type>
             <joint name="${robot_name}_joint7">
-                <hardwareInterface>hardware_interface/PositionJointInterface</hardwareInterface>
+                <hardwareInterface>hardware_interface/${hi}</hardwareInterface>
             </joint>
             <actuator name="${robot_name}_motor_7">
-                <hardwareInterface>hardware_interface/PositionJointInterface</hardwareInterface>
+                <hardwareInterface>hardware_interface/${hi}</hardwareInterface>
                 <mechanicalReduction>1</mechanicalReduction>
             </actuator>
@@ -82,8 +82,8 @@
                 <type>transmission_interface/SimpleTransmission</type>
                 <joint name="${robot_name}_finger_joint1">
-                    <hardwareInterface>hardware_interface/PositionJointInterface</hardwareInterface>
+                    <hardwareInterface>hardware_interface/${hi}</hardwareInterface>
                 </joint>
                 <actuator name="${robot_name}_finger_joint1">
-                    <hardwareInterface>hardware_interface/PositionJointInterface</hardwareInterface>
+                    <hardwareInterface>hardware_interface/${hi}</hardwareInterface>
                     <mechanicalReduction>1</mechanicalReduction>
                 </actuator>
@@ -92,8 +92,8 @@
                 <type>transmission_interface/SimpleTransmission</type>
                 <joint name="${robot_name}_finger_joint2">
-                    <hardwareInterface>hardware_interface/PositionJointInterface</hardwareInterface>
+                    <hardwareInterface>hardware_interface/${hi}</hardwareInterface>
                 </joint>
                 <actuator name="${robot_name}_finger_joint2">
-                    <hardwareInterface>hardware_interface/PositionJointInterface</hardwareInterface>
+                    <hardwareInterface>hardware_interface/${hi}</hardwareInterface>
                     <mechanicalReduction>1</mechanicalReduction>
                 </actuator>

File: mobile_manipulator/robot_description/mmrobot.urdf.xacro (robot description, xacro)
@@ -2,4 +2,5 @@
 <robot xmlns:xacro="http://www.ros.org/wiki/xacro" name="mmrobot_description">
   <xacro:arg name="robot_name" default="mmrobot"/>
+  <xacro:arg name="panda_hi" default="PositionJointInterface"/>
 <!--
   <xacro:include filename="$(find franka_description)/robots/panda_arm.xacro"/>
@@ -17,4 +18,4 @@
   <xacro:hand ns="$(arg robot_name)" rpy="0 0 ${-pi/4}" connected_to="$(arg robot_name)_link8"/>
   <xacro:panda_gazebo robot_name="$(arg robot_name)" />
-  <xacro:panda_transmission robot_name="$(arg robot_name)" load_hand="true"/>
+  <xacro:panda_transmission robot_name="$(arg robot_name)" load_hand="true" hi="$(arg panda_hi)"/>
 </robot>

Commit message: added hand group on moveit package. Modified configuration and launch files. Added examples

File: mobile_manipulator/franka_description/robots/panda.transmission.xacro (robot description, xacro)
@@ -1,5 +1,5 @@
 <?xml version="1.0"?>
 <robot xmlns:xacro="http://www.ros.org/wiki/xacro">
-    <xacro:macro name="panda_transmission" params="robot_name load_hand hi:='PositionJointInterface'">
+    <xacro:macro name="panda_transmission" params="robot_name load_hand hi:='EffortJointInterface'">
         <!-- Load Gazebo lib and set the robot namespace -->
         <gazebo>

File: mobile_manipulator/franka_description/robots/panda_arm_hand.urdf.xacro (robot description, xacro)
@@ -3,14 +3,9 @@
   <xacro:include filename="$(find mobile_manipulator)/franka_description/robots/panda_arm.xacro"/>
   <xacro:include filename="$(find mobile_manipulator)/franka_description/robots/hand.xacro"/>
-  <!-- for simulation -->
   <xacro:include filename="$(find mobile_manipulator)/franka_description/robots/panda.gazebo.xacro"/>
   <xacro:include filename="$(find mobile_manipulator)/franka_description/robots/panda.transmission.xacro"/>
-  <!-- end for simulation -->
-  <!--xacro:panda_arm /-->
-  <!--xacro:hand ns="panda" rpy="0 0 ${-pi/4}" connected_to="panda_link8"/-->
-  <!-- for simulation -->
-  <!--xacro:arg name="robot_name" default="panda"/-->
-  <!--xacro:panda_gazebo robot_name="$(arg robot_name)" /-->
-  <!--xacro:panda_transmission robot_name="$(arg robot_name)" load_hand="true" /-->
-  <!-- end for simulation -->
+<xacro:panda_arm />
+<xacro:hand ns="panda" rpy="0 0 ${-pi/4}" connected_to="panda_link8"/>
+<xacro:panda_gazebo robot_name="$(arg robot_name)" />
+<xacro:panda_transmission robot_name="$(arg robot_name)"/>
 </robot>

File: mobile_manipulator/robot_description/mmrobot.urdf.xacro (robot description, xacro)
@@ -2,13 +2,10 @@
 <robot xmlns:xacro="http://www.ros.org/wiki/xacro" name="mmrobot_description">
   <xacro:arg name="robot_name" default="mmrobot"/>
-  <xacro:arg name="panda_hi" default="PositionJointInterface"/>
-<!--
-  <xacro:include filename="$(find franka_description)/robots/panda_arm.xacro"/>
-  <xacro:include filename="$(find franka_description)/robots/hand.xacro"/>
-  <xacro:include filename="$(find franka_description)/robots/panda.gazebo.xacro"/>
-  <xacro:include filename="$(find franka_description)/robots/panda.transmission.xacro"/>
--->
+  <xacro:arg name="panda_hi" default="EffortJointInterface"/>
+  <xacro:include filename="$(find mobile_manipulator)/franka_description/robots/panda_arm.xacro"/>
+  <xacro:include filename="$(find mobile_manipulator)/franka_description/robots/hand.xacro"/>
+  <xacro:include filename="$(find mobile_manipulator)/franka_description/robots/panda.gazebo.xacro"/>
+  <xacro:include filename="$(find mobile_manipulator)/franka_description/robots/panda.transmission.xacro"/>
   <xacro:include filename="$(find mobile_manipulator)/boxer_description/urdf/boxer.urdf.xacro"/>
-  <xacro:include filename="$(find mobile_manipulator)/franka_description/robots/panda_arm_hand.urdf.xacro"/>
   <!-- Boxer -->
   <xacro:boxer_description/>
@@ -16,6 +13,6 @@
   <!-- Panda Arm -->
   <xacro:panda_arm arm_id='$(arg robot_name)' connected_to='top_mount' xyz='-0.15 0 0' />
-  <xacro:hand ns="$(arg robot_name)" rpy="0 0 ${-pi/4}" connected_to="$(arg robot_name)_link8"/>
+  <xacro:hand ns="mmrobot" rpy="0 0 ${-pi/4}" connected_to="$(arg robot_name)_link8"/>
   <xacro:panda_gazebo robot_name="$(arg robot_name)" />
-  <xacro:panda_transmission robot_name="$(arg robot_name)" load_hand="true" hi="$(arg panda_hi)"/>
+  <xacro:panda_transmission robot_name="$(arg robot_name)" load_hand="true"/>
 </robot>

Commit message: Fixed velocity interface, now loading controllers. Fixed bug with default hi. Now load hand controller only in effort interface

File: mobile_manipulator/franka_description/robots/panda.transmission.xacro (robot description, xacro)
@@ -1,5 +1,5 @@
 <?xml version="1.0"?>
 <robot xmlns:xacro="http://www.ros.org/wiki/xacro">
-    <xacro:macro name="panda_transmission" params="robot_name load_hand hi:='EffortJointInterface'">
+    <xacro:macro name="panda_transmission" params="robot_name load_hand hi">
         <!-- Load Gazebo lib and set the robot namespace -->
         <gazebo>

File: mobile_manipulator/robot_description/mmrobot.urdf.xacro (robot description, xacro)
@@ -13,6 +13,6 @@
   <!-- Panda Arm -->
   <xacro:panda_arm arm_id='$(arg robot_name)' connected_to='top_mount' xyz='-0.15 0 0' />
-  <xacro:hand ns="mmrobot" rpy="0 0 ${-pi/4}" connected_to="$(arg robot_name)_link8"/>
+  <xacro:hand ns='$(arg robot_name)' rpy="0 0 ${-pi/4}" connected_to="$(arg robot_name)_link8"/>
   <xacro:panda_gazebo robot_name="$(arg robot_name)" />
-  <xacro:panda_transmission robot_name="$(arg robot_name)" load_hand="true"/>
+  <xacro:panda_transmission robot_name="$(arg robot_name)" load_hand="true" hi="$(arg panda_hi)"/>
 </robot>
