Commit message: Adds grasp fix option to the panda gazebo setup. It can be set using the parameter grasp_fix. However, it requires two packages to be installed

File: mobile_manipulator/franka_description/robots/panda.gazebo.xacro (robot description, xacro)
@@ -1,5 +1,5 @@
 <?xml version="1.0"?>
 <robot xmlns:xacro="http://www.ros.org/wiki/xacro">
-    <xacro:macro name="panda_gazebo" params="robot_name">
+    <xacro:macro name="panda_gazebo" params="robot_name grasp_fix:='False'">
         <!-- Link0 -->
         <gazebo reference="${robot_name}_link0">
@@ -74,4 +74,25 @@
             <mu2>0.2</mu2>
         </gazebo>
+        <!-- In order to use this grasping fix, two packages are required
+             gazebo-pkgs, general-messages-pkgs-->
+        <xacro:if value="${grasp_fix}">
+          <gazebo>
+             <plugin name="gazebo_grasp_fix" filename="libgazebo_grasp_fix.so">
+                  <arm>
+                     <arm_name>${robot_name}_franka_gripper</arm_name>
+                     <palm_link>${robot_name}_link7</palm_link>
+                     <gripper_link>${robot_name}_leftfinger</gripper_link>
+                     <gripper_link>${robot_name}_rightfinger</gripper_link>
+                  </arm>
+                 <forces_angle_tolerance>100</forces_angle_tolerance>
+                 <update_rate>10</update_rate>
+                 <grip_count_threshold>4</grip_count_threshold>
+                 <max_grip_count>8</max_grip_count>
+                 <release_tolerance>0.0025</release_tolerance>
+                 <disable_collisions_on_attach>false</disable_collisions_on_attach>
+                 <contact_topic>__default_topic__</contact_topic>
+              </plugin>
+          </gazebo>
+        </xacro:if>
     </xacro:macro>
 </robot>

File: mobile_manipulator/franka_description/robots/panda.transmission.xacro (robot description, xacro)
@@ -82,8 +82,8 @@
                 <type>transmission_interface/SimpleTransmission</type>
                 <joint name="${robot_name}_finger_joint1">
-                    <hardwareInterface>hardware_interface/${hi}</hardwareInterface>
+                    <hardwareInterface>hardware_interface/EffortJointInterface</hardwareInterface>
                 </joint>
                 <actuator name="${robot_name}_finger_joint1">
-                    <hardwareInterface>hardware_interface/${hi}</hardwareInterface>
+                    <hardwareInterface>hardware_interface/EffortJointInterface</hardwareInterface>
                     <mechanicalReduction>1</mechanicalReduction>
                 </actuator>
@@ -92,8 +92,8 @@
                 <type>transmission_interface/SimpleTransmission</type>
                 <joint name="${robot_name}_finger_joint2">
-                    <hardwareInterface>hardware_interface/${hi}</hardwareInterface>
+                    <hardwareInterface>hardware_interface/EffortJointInterface</hardwareInterface>
                 </joint>
                 <actuator name="${robot_name}_finger_joint2">
-                    <hardwareInterface>hardware_interface/${hi}</hardwareInterface>
+                    <hardwareInterface>hardware_interface/EffortJointInterface</hardwareInterface>
                     <mechanicalReduction>1</mechanicalReduction>
                 </actuator>

File: mobile_manipulator/robot_description/mmrobot.urdf.xacro (robot description, xacro)
@@ -3,4 +3,5 @@
   <xacro:arg name="robot_name" default="mmrobot"/>
   <xacro:arg name="panda_hi" default="EffortJointInterface"/>
+  <xacro:arg name="grasp_fix" default="False"/>
   <xacro:include filename="$(find mobile_manipulator)/franka_description/robots/panda_arm.xacro"/>
   <xacro:include filename="$(find mobile_manipulator)/franka_description/robots/hand.xacro"/>
@@ -14,5 +15,5 @@
   <xacro:panda_arm arm_id='$(arg robot_name)' connected_to='top_mount' xyz='-0.15 0 0' />
   <xacro:hand ns='$(arg robot_name)' rpy="0 0 ${-pi/4}" connected_to="$(arg robot_name)_link8"/>
-  <xacro:panda_gazebo robot_name="$(arg robot_name)" />
+  <xacro:panda_gazebo robot_name="$(arg robot_name)" grasp_fix="$(arg grasp_fix)" />
   <xacro:panda_transmission robot_name="$(arg robot_name)" load_hand="true" hi="$(arg panda_hi)"/>
 </robot>
