Commit message: Resolves issue of dependency to CAD files of franka_description

File: mobile_manipulator/franka_description/robots/hand.xacro (robot description, xacro)
@@ -12,10 +12,10 @@
       <visual>
         <geometry>
-          <mesh filename="package://franka_description/meshes/visual/hand.dae"/>
+          <mesh filename="package://mobile_manipulator/franka_description/meshes/visual/hand.dae"/>
         </geometry>
       </visual>
       <collision>
         <geometry>
-          <mesh filename="package://franka_description/meshes/collision/hand.stl"/>
+          <mesh filename="package://mobile_manipulator/franka_description/meshes/collision/hand.stl"/>
         </geometry>
       </collision>
@@ -31,10 +31,10 @@
       <visual>
         <geometry>
-          <mesh filename="package://franka_description/meshes/visual/finger.dae"/>
+          <mesh filename="package://mobile_manipulator/franka_description/meshes/visual/finger.dae"/>
         </geometry>
       </visual>
       <collision>
         <geometry>
-          <mesh filename="package://franka_description/meshes/collision/finger.stl"/>
+          <mesh filename="package://mobile_manipulator/franka_description/meshes/collision/finger.stl"/>
         </geometry>
       </collision>
@@ -51,5 +51,5 @@
         <origin xyz="0 0 0" rpy="0 0 ${pi}"/>
         <geometry>
-          <mesh filename="package://franka_description/meshes/visual/finger.dae"/>
+          <mesh filename="package://mobile_manipulator/franka_description/meshes/visual/finger.dae"/>
         </geometry>
       </visual>
@@ -57,5 +57,5 @@
         <origin xyz="0 0 0" rpy="0 0 ${pi}"/>
         <geometry>
-          <mesh filename="package://franka_description/meshes/collision/finger.stl"/>
+          <mesh filename="package://mobile_manipulator/franka_description/meshes/collision/finger.stl"/>
         </geometry>
       </collision>

File: mobile_manipulator/franka_description/robots/panda_arm.xacro (robot description, xacro)
@@ -1,5 +1,5 @@
 <?xml version='1.0' encoding='utf-8'?>
 <robot xmlns:xacro="http://www.ros.org/wiki/xacro" name="panda">
-  <xacro:macro name="panda_arm" params="arm_id:='panda' description_pkg:='franka_description' connected_to:='' xyz:='0 0 0' rpy:='0 0 0'">
+  <xacro:macro name="panda_arm" params="arm_id:='panda' description_pkg:='mobile_manipulator/franka_description' connected_to:='' xyz:='0 0 0' rpy:='0 0 0'">
     <xacro:unless value="${not connected_to}">
       <joint name="${arm_id}_joint_${connected_to}" type="fixed">

Commit message: Add virtual link for the end effector, link in the center of both fingers

File: mobile_manipulator/franka_description/robots/hand.xacro (robot description, xacro)
@@ -28,4 +28,5 @@
       <!-- end for simulation -->
     </link>
+    <link name="${ns}_ee"/>
     <link name="${ns}_leftfinger">
       <visual>
@@ -68,4 +69,9 @@
       <!-- end for simulation -->
     </link>
+    <joint name="${ns}_ee_joint" type="fixed">
+      <parent link="${ns}_hand"/>
+      <child link="${ns}_ee"/>
+      <origin xyz="0 0 0.1" rpy="0 0 0"/>
+    </joint>
     <joint name="${ns}_finger_joint1" type="prismatic">
       <parent link="${ns}_hand"/>
