Commit message: Cleanup for master branches
Merges boxer_custom_description and boxer_description to remove
duplicates. In this process, meshes are moved to
boxer_description/meshes.

File: mobile_manipulator/boxer_description/urdf/boxer.gazebo.xacro (robot description, xacro)
@@ -298,6 +298,4 @@
       <minDepth>0.0</minDepth>
     </gazebo>
-    <!-- Load the main robot description -->
-    <!-- <xacro:include filename="$(find boxer_description)/urdf/boxer.urdf.xacro"/> -->
   </xacro:macro>
 </robot>

File: mobile_manipulator/boxer_description/urdf/boxer.xacro (robot description, xacro)
@@ -1,5 +1,5 @@
 <?xml version="1.0"?>
 <robot name="boxer_description" xmlns:xacro="http://www.ros.org/wiki/xacro">
-	<xacro:include filename="$(find mobile_manipulator)/boxer_custom_description/urdf/materials.urdf.xacro"/>
+	<xacro:include filename="$(find mobile_manipulator)/boxer_description/urdf/materials.urdf.xacro"/>
 	<xacro:macro name="boxer_description">
 		<link name="chassis_link">
@@ -12,5 +12,5 @@
 				<origin xyz="0 0 0" rpy="0 0 0" />
 				<geometry>
-					<mesh filename="package://mobile_manipulator/boxer_custom_description/meshes/chassis_link.dae" />
+					<mesh filename="package://mobile_manipulator/boxer_description/meshes/chassis_link.dae" />
 				</geometry>
 				<material name="">
@@ -21,5 +21,5 @@
 				<origin xyz="0 0 0" rpy="0 0 0" />
 				<geometry>
-					<mesh filename="package://mobile_manipulator/boxer_custom_description/meshes/chassis_link.STL" />
+					<mesh filename="package://mobile_manipulator/boxer_description/meshes/chassis_link.STL" />
 				</geometry>
 			</collision>
@@ -34,5 +34,5 @@
 				<origin xyz="0 0 0" rpy="0 0 0" />
 				<geometry>
-					<mesh filename="package://mobile_manipulator/boxer_custom_description/meshes/internal_link.dae" />
+					<mesh filename="package://mobile_manipulator/boxer_description/meshes/internal_link.dae" />
 				</geometry>
 				<material name="Boxer_DarkGrey"/>
@@ -44,5 +44,5 @@
       <!-- (The z axis is scaled since the whole model is rotated at the joint, and collision model resolution isn't
       very smart.) -->
-      <mesh filename="package://mobile_manipulator/boxer_custom_description/meshes/internal_link.STL" />
+      <mesh filename="package://mobile_manipulator/boxer_description/meshes/internal_link.STL" />
   </geometry>
 </collision>
@@ -63,5 +63,5 @@
 		<origin xyz="0 0 0" rpy="0 0 0" />
 		<geometry>
-			<mesh filename="package://mobile_manipulator/boxer_custom_description/meshes/lift_link.dae" />
+			<mesh filename="package://mobile_manipulator/boxer_description/meshes/lift_link.dae" />
 		</geometry>
 		<material name="">
@@ -72,5 +72,5 @@
 		<origin xyz="0 0 0" rpy="0 0 0" />
 		<geometry>
-			<mesh filename="package://mobile_manipulator/boxer_custom_description/meshes/lift_link.STL" />
+			<mesh filename="package://mobile_manipulator/boxer_description/meshes/lift_link.STL" />
 		</geometry>
 	</collision>
@@ -88,12 +88,12 @@
 		<origin xyz="0 0 0" rpy="0 0 0" />
 		<geometry>
-			<mesh filename="package://mobile_manipulator/boxer_custom_description/meshes/top_plate.stl" />
-		</geometry>
-		<material name="Boxer_DarkGrey" />
-	</visual>
-	<collision>
-		<origin xyz="0 0 0" rpy="0 0 0" />
-		<geometry>
-			<mesh filename="package://mobile_manipulator/boxer_custom_description/meshes/top_plate_collision.stl" />
+			<mesh filename="package://mobile_manipulator/boxer_description/meshes/top_plate.stl" />
+		</geometry>
+		<material name="Boxer_DarkGrey" />
+	</visual>
+	<collision>
+		<origin xyz="0 0 0" rpy="0 0 0" />
+		<geometry>
+			<mesh filename="package://mobile_manipulator/boxer_description/meshes/top_plate_collision.stl" />
 		</geometry>
 	</collision>
@@ -108,12 +108,12 @@
 		<origin xyz="0 0 0" rpy="0 0 0" />
 		<geometry>
-			<mesh filename="package://mobile_manipulator/boxer_custom_description/meshes/extrusion.stl" />
-		</geometry>
-		<material name="Boxer_DarkGrey" />
-	</visual>
-	<collision>
-		<origin xyz="0 0 0" rpy="0 0 0" />
-		<geometry>
-			<mesh filename="package://mobile_manipulator/boxer_custom_description/meshes/extrusion.stl" />
+			<mesh filename="package://mobile_manipulator/boxer_description/meshes/extrusion.stl" />
+		</geometry>
+		<material name="Boxer_DarkGrey" />
+	</visual>
+	<collision>
+		<origin xyz="0 0 0" rpy="0 0 0" />
+		<geometry>
+			<mesh filename="package://mobile_manipulator/boxer_description/meshes/extrusion.stl" />
 		</geometry>
 	</collision>
@@ -128,12 +128,12 @@
 		<origin xyz="0 0 0" rpy="0 0 0" />
 		<geometry>
-			<mesh filename="package://mobile_manipulator/boxer_custom_description/meshes/extrusion.stl" />
-		</geometry>
-		<material name="Boxer_DarkGrey" />
-	</visual>
-	<collision>
-		<origin xyz="0 0 0" rpy="0 0 0" />
-		<geometry>
-			<mesh filename="package://mobile_manipulator/boxer_custom_description/meshes/extrusion.stl" />
+			<mesh filename="package://mobile_manipulator/boxer_description/meshes/extrusion.stl" />
+		</geometry>
+		<material name="Boxer_DarkGrey" />
+	</visual>
+	<collision>
+		<origin xyz="0 0 0" rpy="0 0 0" />
+		<geometry>
+			<mesh filename="package://mobile_manipulator/boxer_description/meshes/extrusion.stl" />
 		</geometry>
 	</collision>
@@ -148,12 +148,12 @@
 		<origin xyz="0 0 0" rpy="0 0 0" />
 		<geometry>
-			<mesh filename="package://mobile_manipulator/boxer_custom_description/meshes/extrusion.stl" />
-		</geometry>
-		<material name="Boxer_DarkGrey" />
-	</visual>
-	<collision>
-		<origin xyz="0 0 0" rpy="0 0 0" />
-		<geometry>
-			<mesh filename="package://mobile_manipulator/boxer_custom_description/meshes/extrusion.stl" />
+			<mesh filename="package://mobile_manipulator/boxer_description/meshes/extrusion.stl" />
+		</geometry>
+		<material name="Boxer_DarkGrey" />
+	</visual>
+	<collision>
+		<origin xyz="0 0 0" rpy="0 0 0" />
+		<geometry>
+			<mesh filename="package://mobile_manipulator/boxer_description/meshes/extrusion.stl" />
 		</geometry>
 	</collision>
@@ -168,12 +168,12 @@
 		<origin xyz="0 0 0" rpy="0 0 0" />
 		<geometry>
-			<mesh filename="package://mobile_manipulator/boxer_custom_description/meshes/extrusion.stl" />
-		</geometry>
-		<material name="Boxer_DarkGrey" />
-	</visual>
-	<collision>
-		<origin xyz="0 0 0" rpy="0 0 0" />
-		<geometry>
-			<mesh filename="package://mobile_manipulator/boxer_custom_description/meshes/extrusion.stl" />
+			<mesh filename="package://mobile_manipulator/boxer_description/meshes/extrusion.stl" />
+		</geometry>
+		<material name="Boxer_DarkGrey" />
+	</visual>
+	<collision>
+		<origin xyz="0 0 0" rpy="0 0 0" />
+		<geometry>
+			<mesh filename="package://mobile_manipulator/boxer_description/meshes/extrusion.stl" />
 		</geometry>
 	</collision>
@@ -188,12 +188,12 @@
 		<origin xyz="0 0 0" rpy="0 0 0" />
 		<geometry>
-			<mesh filename="package://mobile_manipulator/boxer_custom_description/meshes/top_plate.stl" />
-		</geometry>
-		<material name="Boxer_DarkGrey" />
-	</visual>
-	<collision>
-		<origin xyz="0 0 0" rpy="0 0 0" />
-		<geometry>
-			<mesh filename="package://mobile_manipulator/boxer_custom_description/meshes/top_plate_collision.stl" />
+			<mesh filename="package://mobile_manipulator/boxer_description/meshes/top_plate.stl" />
+		</geometry>
+		<material name="Boxer_DarkGrey" />
+	</visual>
+	<collision>
+		<origin xyz="0 0 0" rpy="0 0 0" />
+		<geometry>
+			<mesh filename="package://mobile_manipulator/boxer_description/meshes/top_plate_collision.stl" />
 		</geometry>
 	</collision>
@@ -327,7 +327,7 @@
 <link name="base_footprint" />
 <joint name="base_footprint_joint" type="fixed">
-	<origin xyz="0 0 0.08" rpy="0 0 0" />
-	<parent link="base_footprint" />
-	<child link="base_link" />
+	<origin xyz="0 0 -0.08" rpy="0 0 0" />
+	<parent link="base_link" />
+	<child link="base_footprint" />
 </joint>
 <!-- Link for the position of the laser. -->
@@ -405,4 +405,3 @@
 </joint>
 </xacro:macro>
-<xacro:include filename="$(optenv BOXER_URDF_EXTRAS empty.urdf)" />
 </robot>

File: mobile_manipulator/robot_description/boxer.urdf.xacro (robot description, xacro)
@@ -2,5 +2,5 @@
 <robot xmlns:xacro="http://www.ros.org/wiki/xacro" name="boxer_description">
   <xacro:arg name="robot_name" default="boxer"/>
-  <xacro:include filename="$(find mobile_manipulator)/boxer_description/boxer.urdf.xacro"/>
+  <xacro:include filename="$(find mobile_manipulator)/boxer_description/urdf/boxer.urdf.xacro"/>
   <!-- Boxer -->
   <xacro:boxer_description/>

File: mobile_manipulator/robot_description/mmrobot.urdf.xacro (robot description, xacro)
@@ -9,5 +9,5 @@
   <xacro:include filename="$(find franka_description)/robots/panda.transmission.xacro"/>
 -->
-  <xacro:include filename="$(find mobile_manipulator)/boxer_description/boxer.urdf.xacro"/>
+  <xacro:include filename="$(find mobile_manipulator)/boxer_description/urdf/boxer.urdf.xacro"/>
   <xacro:include filename="$(find mobile_manipulator)/franka_description/robots/panda_arm_hand.urdf.xacro"/>
   <!-- Boxer -->

Commit message: Adds 3D camera integration into the gazebo files. The camera is mounted onto the topmount of the boxer base

File: mobile_manipulator/boxer_description/urdf/boxer.gazebo.xacro (robot description, xacro)
@@ -183,5 +183,5 @@
       </sensor>
     </gazebo>
-    <gazebo reference="stereo_left">
+    <!--gazebo reference="stereo_left">
       <material>Gazebo/Grey</material>
       <sensor type="camera" name="camera_left">
@@ -220,5 +220,5 @@
         </plugin>
       </sensor>
-    </gazebo>
+    </gazebo-->
     <!-- Right -->
     <!--gazebo reference="stereo_right">
@@ -260,4 +260,46 @@
       </sensor>
     </gazebo-->
+    <gazebo reference="top_camera">
+      <sensor name="top_camera" type="depth">
+        <update_rate>20</update_rate>
+        <camera>
+          <horizontal_fov>1.047198</horizontal_fov>
+          <image>
+            <width>640</width>
+            <height>480</height>
+            <format>R8G8B8</format>
+          </image>
+          <clip>
+            <near>0.05</near>
+            <far>3</far>
+          </clip>
+        </camera>
+        <plugin name="depth_camera_controller" filename="libgazebo_ros_openni_kinect.so">
+          <baseline>0.2</baseline>
+          <alwaysOn>true</alwaysOn>
+          <updateRate>1.0</updateRate>
+          <cameraName>depth_camera_ir</cameraName>
+          <imageTopicName>/depth_camera/color/image_raw</imageTopicName>
+          <cameraInfoTopicName>/depth_camera/color/camera_info</cameraInfoTopicName>
+          <depthImageTopicName>/depth_camera/depth/image_raw</depthImageTopicName>
+          <depthImageInfoTopicName>/depth_camera/depth/camera_info</depthImageInfoTopicName>
+          <pointCloudTopicName>/depth_camera/depth/points</pointCloudTopicName>
+          <robotNamespace>/</robotNamespace>
+          <frameName>depth_camera</frameName>
+          <pointCloudCutoff>0.5</pointCloudCutoff>
+          <pointCloudCutoffMax>3.0</pointCloudCutoffMax>
+          <distortionK1>0.00000001</distortionK1>
+          <distortionK2>0.00000001</distortionK2>
+          <distortionK3>0.00000001</distortionK3>
+          <distortionT1>0.00000001</distortionT1>
+          <distortionT2>0.00000001</distortionT2>
+          <CxPrime>0</CxPrime>
+          <Cx>0</Cx>
+          <Cy>0</Cy>
+          <focalLength>0</focalLength>
+          <hackBaseline>0</hackBaseline>
+        </plugin>
+      </sensor>
+    </gazebo>
     <xacro:macro name="wheel" params="side">
       <gazebo reference="wheel_${side}_link">

File: mobile_manipulator/boxer_description/urdf/boxer.xacro (robot description, xacro)
@@ -358,4 +358,16 @@
 	<child link="stereo_right" />
 </joint>
+<link name="top_camera" />
+<joint name="top_camera_joint" type="fixed">
+	<origin xyz="0.1 0 0.1" rpy="0 0 0" />
+	<parent link="top_mount" />
+	<child link="top_camera" />
+</joint>
+<link name="depth_camera" />
+<joint name="depth_camera_joint" type="fixed">
+	<origin xyz="0.1 0 0.1" rpy="${-pi/2} 0 ${-pi/2}" />
+	<parent link="top_camera" />
+	<child link="depth_camera" />
+</joint>
 <!-- Sonar links to base link joints -->
 <link name="rear_left_sonar_link" />
