Commit message: Minor Modifications of URDF
Adds virtual links to the robot for collision avoidance.
Changes spheres from mesh to gazebo internal sphere.
Updates joystick control to spin on base motion.
Adds parameters to octomap launch to allow loading of a prerecorded map.

File: mobile_manipulator/boxer_description/urdf/boxer.xacro (robot description, xacro)
@@ -323,4 +323,11 @@
 	<child link="chassis_link" />
 </joint>
+<!-- link for collision avoidance-->
+<link name="base_sphere" />
+<joint name="base_sphere_joint=" type="fixed">
+  <origin xyz="0.15 0 0.25" />
+  <parent link="base_link" />
+  <child link="base_sphere" />
+</joint>
 <!-- Projection of base_link on the ground to get the 3D data
 in the right frame w.r.t the ground. -->
@@ -360,5 +367,5 @@
 <link name="top_camera" />
 <joint name="top_camera_joint" type="fixed">
-	<origin xyz="0.1 0 0.1" rpy="0 0 0" />
+	<origin xyz="0.1 0 0.3" rpy="0 ${-0/10} 0" />
 	<parent link="top_mount" />
 	<child link="top_camera" />

File: mobile_manipulator/franka_description/robots/panda_arm.xacro (robot description, xacro)
@@ -99,4 +99,11 @@
       <!-- end for simulation -->
     </joint>
+    <!-- sphere 2 for collision avoidance-->
+    <link name="${arm_id}_link2_sphere" />
+    <joint name="${arm_id}_link2_sphere_joint" type="fixed">
+      <origin xyz="0 -0.1896 0"/>
+      <parent link="${arm_id}_link2"/>
+      <child link="${arm_id}_link2_sphere"/>
+    </joint>
     <link name="${arm_id}_link3">
       <visual>
@@ -249,4 +256,11 @@
       <!-- end for simulation -->
     </joint>
+    <!-- sphere 7 for collision avoidance-->
+    <link name="${arm_id}_link7_sphere" />
+    <joint name="${arm_id}_link7_sphere_joint" type="fixed">
+      <origin xyz="0 0 0"/>
+      <parent link="${arm_id}_link7"/>
+      <child link="${arm_id}_link7_sphere"/>
+    </joint>
     <link name="${arm_id}_link8">
       <!-- for simulation -->

File: mobile_manipulator/world/urdf/sphere.xacro (robot description, xacro)
@@ -11,5 +11,5 @@
       <origin xyz="0 0 0" rpy="0 0 0"/>
       <geometry>
-        <mesh filename="package://mobile_manipulator/world/meshes/sphere.dae" scale="${r} ${r} ${r}"/>
+        <sphere radius="${r/100}"/>
       </geometry>
       <material name="Gray" />
@@ -18,5 +18,5 @@
       <origin xyz="0 0 0" rpy="0 0 0"/>
       <geometry>
-        <mesh filename="package://mobile_manipulator/world/meshes/sphere.dae"/>
+        <sphere radius="${r/100}"/>
       </geometry>
     </collision>
