Commit message: Adds primitive shapes

File: mobile_manipulator/world/urdf/box.xacro (robot description, xacro)
@@ -1,6 +1,6 @@
 <?xml version="1.0"?>
 <robot name="robot" xmlns:xacro="http://www.ros.org/wiki/xacro">
-  <xacro:macro name="spawn_sphere" params="sphere_name:='sphere_0' r:='1' xyz:='0 0 0' rpy:='0 0 0' color:='Gray'">
-  <link name="${sphere_name}">
+  <xacro:macro name="spawn_box" params="box_name:='box_0' b:='1' l:='1' h:='1' xyz:='0 0 0' rpy:='0 0 0.785' color:='White'">
+  <link name="${box_name}">
     <inertial>
       <origin xyz="0 0 0" rpy="0 0 0"/>
@@ -11,21 +11,21 @@
       <origin xyz="0 0 0" rpy="0 0 0"/>
       <geometry>
-        <sphere radius="${r/100}"/>
+        <box size="${b} ${l} ${h}" />
       </geometry>
-      <material name="${color}" />
+      <material name="Gray" />
     </visual>
     <collision>
       <origin xyz="0 0 0" rpy="0 0 0"/>
       <geometry>
-        <sphere radius="${r/100}"/>
+        <box size="${b} ${l} ${h}" />
       </geometry>
     </collision>
   </link>
-  <joint name="world_${sphere_name}_joint" type="fixed">
+  <joint name="world_${box_name}_joint" type="fixed">
     <origin xyz="${xyz}" rpy="${rpy}"/>
     <parent link="world"/>
-    <child link="${sphere_name}"/>
+    <child link="${box_name}"/>
   </joint>
-  <gazebo reference="${sphere_name}">
+  <gazebo reference="${box_name}">
     <material>Gazebo/${color}</material>
   </gazebo>

File: mobile_manipulator/world/urdf/cylinder.xacro (robot description, xacro)
@@ -1,6 +1,6 @@
 <?xml version="1.0"?>
 <robot name="robot" xmlns:xacro="http://www.ros.org/wiki/xacro">
-  <xacro:macro name="spawn_sphere" params="sphere_name:='sphere_0' r:='1' xyz:='0 0 0' rpy:='0 0 0' color:='Gray'">
-  <link name="${sphere_name}">
+  <xacro:macro name="spawn_cylinder" params="cylinder_name:='cylinder_0' r:='1' l:='100' xyz:='0 0 0' rpy:='0 0 0' color:='Gray'">
+  <link name="${cylinder_name}">
     <inertial>
       <origin xyz="0 0 0" rpy="0 0 0"/>
@@ -11,5 +11,5 @@
       <origin xyz="0 0 0" rpy="0 0 0"/>
       <geometry>
-        <sphere radius="${r/100}"/>
+        <cylinder radius="${r/100}" length="${l/100}"/>
       </geometry>
       <material name="${color}" />
@@ -18,14 +18,14 @@
       <origin xyz="0 0 0" rpy="0 0 0"/>
       <geometry>
-        <sphere radius="${r/100}"/>
+        <cylinder radius="${r/100}" length="${l/100}"/>
       </geometry>
     </collision>
   </link>
-  <joint name="world_${sphere_name}_joint" type="fixed">
+  <joint name="world_${cylinder_name}_joint" type="fixed">
     <origin xyz="${xyz}" rpy="${rpy}"/>
     <parent link="world"/>
-    <child link="${sphere_name}"/>
+    <child link="${cylinder_name}"/>
   </joint>
-  <gazebo reference="${sphere_name}">
+  <gazebo reference="${cylinder_name}">
     <material>Gazebo/${color}</material>
   </gazebo>
